Commit message: Modify launch file and map file, TF publisher file

File: src/nav2_px4/urdf/x500.urdf (robot description, URDF)
Before this commit: robot x500, 9 links, 8 joints
Links:
- removed link gps_link
- added link x500_lidar_2d_0/base_link/navsat_sensor, mass 0.001
Joints:
- joint gps_joint: child gps_link -> x500_lidar_2d_0/base_link/navsat_sensor

Commit message: Add RTAB-MAP and PX4 Integration

File: src/nav2_px4/urdf/x500.urdf (robot description, URDF)
Before this commit: robot x500, 9 links, 8 joints
Links:
- link body: geometry collision box size=0.015 0.015 0.21; collision box size=0.015 0.015 0.21
- link rotor_0: geometry collision box size=0.2792307692307692 0.016923076923076923 0.00084615384615384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; visual mesh filename=package://nav2_px4/meshes/1345_prop_ccw.stl scale=0.8461538461538461 0.8461538461538461 0.8461538461538461
- link rotor_1: geometry collision box size=0.2792307692307692 0.016923076923076923 0.00084615384615384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; visual mesh filename=package://nav2_px4/meshes/1345_prop_ccw.stl scale=0.8461538461538461 0.8461538461538461 0.8461538461538461
- link rotor_2: geometry collision box size=0.2792307692307692 0.016923076923076923 0.00084615384615384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; visual mesh filename=package://nav2_px4/meshes/1345_prop_cw.stl scale=0.8461538461538461 0.8461538461538461 0.8461538461538461
- link rotor_3: geometry collision box size=0.2792307692307692 0.016923076923076923 0.00084615384615384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; visual mesh filename=package://nav2_px4/meshes/1345_prop_cw.stl scale=0.8461538461538461 0.8461538461538461 0.8461538461538461
- link x500_lidar_2d_0/link/lidar_2d_v2: geometry collision box size=0.056 0.056 0.018; collision box size=0.06 0.06 0.041
