Commit message: Add rtabmap codes

File: src/rtabmap_nav2_px4/urdf/x500_rtab.urdf (robot description, URDF)
Before this commit: robot x500, 13 links, 12 joints
Links:
- link body: geometry collision box size=0.015 0.015 0.21; collision box size=0.015 0.015 0.21
- link rotor_0: geometry collision box size=0.2792307692307692 0.016923076923076923 0.00084615384615384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; visual mesh filename=package://rtabmap_nav2_px4/meshes/1345_prop_ccw.stl scale=0.8461538461538461 0.8461538461538461 0.8461538461538461
- link rotor_1: geometry collision box size=0.2792307692307692 0.016923076923076923 0.00084615384615384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; visual mesh filename=package://rtabmap_nav2_px4/meshes/1345_prop_ccw.stl scale=0.8461538461538461 0.8461538461538461 0.8461538461538461
- link rotor_2: geometry collision box size=0.2792307692307692 0.016923076923076923 0.00084615384615384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; visual mesh filename=package://rtabmap_nav2_px4/meshes/1345_prop_cw.stl scale=0.8461538461538461 0.8461538461538461 0.8461538461538461
- link rotor_3: geometry collision box size=0.2792307692307692 0.016923076923076923 0.00084615384615384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; visual mesh filename=package://rtabmap_nav2_px4/meshes/1345_prop_cw.stl scale=0.8461538461538461 0.8461538461538461 0.8461538461538461
- link x500_rtab_0/OakD-Lite/base_link/IMX214: geometry collision box size=0.0175 0.091 0.028; visual mesh filename=package://rtabmap_nav2_px4/meshes/OakDLite.dae scale=1 1 1
- link x500_rtab_0/link/lidar_2d_v2: geometry collision box size=0.056 0.056 0.018; collision box size=0.06 0.06 0.041
